File: ICE40-DAC_Rev_A.kicad_pcb (KiCad board)
At the start: 2 copper layers, 30 x 50 mm, 51 parts, among them Q1 NA(BC817-40(SOT-23)), U1 THS5641AIDW(SOIC28), U2 SN74ACT244DWR(SOIC-20)

Commit message: Update
Updated trace names
Connections:
- net /LED1 renamed /GPIO_Pin<10>
- net /LED2 renamed /GPIO_Pin<12>
- net /PIO2_1 renamed /GPIO_Pin<30>
- net /PIO2_2 renamed /GPIO_Pin<28>
- net /PIO2_3 renamed /GPIO_Pin<26>
- net /PIO2_4 renamed /GPIO_Pin<24>
- net /PIO2_5 renamed /GPIO_Pin<22>
- net /PIO2_6 renamed /GPIO_Pin<20>
- net /PIO2_7 renamed /GPIO_Pin<18>
- net /PIO2_8/TxD renamed /GPIO_Pin<16>
- net /PIO2_9/RxD renamed /GPIO_Pin<14>
- net /PIO3_10A renamed /GPIO_Pin<31>
- net /PIO3_10B renamed /GPIO_Pin<33>
- net /PIO3_12A renamed /GPIO_Pin<34>
- net /PIO3_12B renamed /GPIO_Pin<32>
- net /PIO3_1A renamed /DAC_D0
- net /PIO3_1B renamed /DAC_D1
- net /PIO3_2A renamed /DAC_D2
- net /PIO3_2B renamed /DAC_D3
- net /PIO3_3A renamed /DAC_D4
- net /PIO3_3B renamed /DAC_D5
- net /PIO3_5A renamed /DAC_D6
- net /PIO3_5B renamed /DAC_D7
- net /PIO3_6A renamed /GPIO_Pin<21>
- net /PIO3_6B renamed /GPIO_Pin<23>
- net /PIO3_7B renamed /GPIO_Pin<25>
- net /PIO3_8A renamed /GPIO_Pin<27>
- net /PIO3_8B renamed /GPIO_Pin<29>
